File: Eagle/projects/DSS_v3/dss_v3.brd (EAGLE design)
At the start: 50 x 90 mm, 59 parts, among them IC1 MC34063AD, IC2 Atmega8a, IC3 TL431, SW1 EC12E_SW, T1 BC846

Commit message: Update dss_v3.brd
Parts:
- removed LED1: BA56-12EWA, 3DIG_7SEG:BX56-12
- removed U$2: (no value), logo:MUELLTONNE_10.00
- added DISP: BA56-12EWA, 3DIG_7SEG:BX56-12
- J1: value (none) -> 12-24V
- LED2: value (none) -> RED
- LED3: value (none) -> GREEN
- X1: value (none) -> PS2
- moved U$3 31.6 mm to (12.2, 30.2)
- moved U$1 12.4 mm to (10.0, 3.75)
- moved C9 8.00 mm to (25.4, 9.95)
- moved C4 7.55 mm to (7.80, 13.4)
- moved C11 7.00 mm to (26.2, 26.5)
- moved C12 7.00 mm to (41.2, 27.8)
- moved C2 7.00 mm to (5.90, 29.3)
- moved R12 7.00 mm to (10.1, 31.7)
- moved R9 7.00 mm to (10.1, 29.3)
- moved SV1 7.00 mm to (38.9, 9.69)
- moved BUZZER_5V_GEN 7.00 mm to (43.4, 51.7)
- moved C1 7.00 mm to (23.3, 72.0)
- moved C14 7.00 mm to (44.7, 22.9)
- moved C3 7.00 mm to (7.77, 17.3)
- moved C6 7.00 mm to (30.6, 61.9)
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Connections:
- net MEGA2: now also DISP.9; no longer LED1.9
- net MEGA31: now also DISP.8; no longer LED1.8
- net MEGA7: now also DISP.12; no longer LED1.12
- net N$1: now also DISP.11; no longer LED1.11
- net N$12: now also DISP.2; no longer LED1.2
- net N$14: now also DISP.1; no longer LED1.1
- net N$19: now also DISP.10; no longer LED1.10
- net N$20: now also DISP.5; no longer LED1.5
- net N$21: now also DISP.3; no longer LED1.3
- net N$3: now also DISP.7; no longer LED1.7
- net N$4: now also DISP.4; no longer LED1.4
Routing:
- net HTR-: track 93.5 -> 38.4 mm, vias 30 -> 12
- net MEGA32: track 65.7 -> 58.9 mm
- net N$6: track 14.2 -> 18.7 mm
- net GND: track 365.6 -> 361.8 mm
- net N$9: track 17.6 -> 13.8 mm
- net MEGA11: track 26.2 -> 29.7 mm
- net MEGA30: track 68.5 -> 66.5 mm
- net M16_MISO: track 44.7 -> 45.9 mm
- net MEGA1: track 51.6 -> 52.8 mm
- net N$5: track 38.1 -> 39.3 mm
- net SH: track 14.2 -> 14.8 mm
Other:
- board size 50 x 90 mm -> 50 x 83 mm

Commit message: update
Parts:
- C6: value 92pf -> 140pf
- L1: value 100uH/250mA -> 210uH/250mA
- R15: value 0.75R -> 1R
Changed lines of the file:
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@@
 <attribute name="VALUE" x="10.34" y="16.555" size="1.27" layer="27" rot="R180"/>
 </element>
-<element name="C6" library="rcl" package="C0805" value="92pf" x="30.64" y="61.89" smashed="yes" rot="MR180">
+<element name="C6" library="rcl" package="C0805" value="140pf" x="30.64" y="61.89" smashed="yes" rot="MR180">
 <attribute name="NAME" x="29.37" y="60.62" size="1.27" layer="26" rot="MR180"/>
 <attribute name="VALUE" x="28.87" y="60.68" size="1.27" layer="28" rot="MR180"/>
@@
 <attribute name="VALUE" x="44.41" y="82.43" size="1.27" layer="28" rot="MR270"/>
 </element>
-<element name="L1" library="eagle-ltspice" library_urn="urn:adsk.eagle:library:217" package="L4532P" package3d_urn="urn:adsk.eagle:package:13289/1" value="100uH/250mA" x="28.02" y="73.64" smashed="yes" rot="MR0">
+<element name="L1" library="eagle-ltspice" library_urn="urn:adsk.eagle:library:217" package="L4532P" package3d_urn="urn:adsk.eagle:package:13289/1" value="210uH/250mA" x="28.02" y="73.64" smashed="yes" rot="MR0">
 <attribute name="NAME" x="28.675" y="76.18" size="1.27" layer="26" rot="MR0"/>
 <attribute name="SPICEMODEL" value="NONE" x="-34.21" y="33" size="1.778" layer="28" rot="MR0" display="off"/>
@@
 <attribute name="VALUE" x="20.64" y="60.68" size="1.27" layer="28" rot="MR180"/>
 </element>
-<element name="R15" library="rcl" package="R0805" value="0.75R" x="20.19" y="66.39" smashed="yes" rot="MR270">
+<element name="R15" library="rcl" package="R0805" value="1R" x="20.19" y="66.39" smashed="yes" rot="MR270">
 <attribute name="NAME" x="18.92" y="67.91" size="1.27" layer="26" rot="MR270"/>
 <attribute name="VALUE" x="17.77" y="63.84" size="1.27" layer="28" rot="MR90"/>

Commit message: update
Parts:
- L1: value 210uH/250mA -> 220uH/250mA
Changed lines of the file:
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@@
 <attribute name="VALUE" x="44.41" y="82.43" size="1.27" layer="28" rot="MR270"/>
 </element>
-<element name="L1" library="eagle-ltspice" library_urn="urn:adsk.eagle:library:217" package="L4532P" package3d_urn="urn:adsk.eagle:package:13289/1" value="210uH/250mA" x="28.02" y="73.64" smashed="yes" rot="MR0">
+<element name="L1" library="eagle-ltspice" library_urn="urn:adsk.eagle:library:217" package="L4532P" package3d_urn="urn:adsk.eagle:package:13289/1" value="220uH/250mA" x="28.02" y="73.64" smashed="yes" rot="MR0">
 <attribute name="NAME" x="28.675" y="76.18" size="1.27" layer="26" rot="MR0"/>
 <attribute name="SPICEMODEL" value="NONE" x="-34.21" y="33" size="1.778" layer="28" rot="MR0" display="off"/>

Commit message: update
Parts:
- C4: device rcl:CT6032 -> rcl:CT3528
- C6: value 140pf -> 154pf
Routing:
- net GND: track 361.8 -> 362.9 mm
